File: FPGA_Lattice_Replica_Icezum/FPGA.sch (KiCad schematic (older format))
At the start: 33 parts, among them U1 iCE40HX1K-TQ144, U2 N25Q032A

Commit message: se corrigieron errores de huellas y referencias que genereban errores cuando se hacia el diseño PCB
Parts:
- LD10: symbol Device:LED -> icezum:LED
Connections:
- net +3V3: now also LD10.A; no longer LD10.2 (A)
- net at R46.2: now also LD10.K; no longer LD10.1 (K)
Changed lines of the file:
@@
 $EndComp
 $Comp
-L Device:LED LD10
+L icezum:LED LD10
 U 1 1 5CFF3FED
-P 5150 7000
-F 0 "LD10" H 5143 6745 50  0000 C CNN
-F 1 "Yellow" H 5143 6836 50  0000 C CNN
-F 2 "footprints:LED_0603" H 5150 7000 50  0001 C CNN
-F 3 "~" H 5150 7000 50  0001 C CNN
-	1    5150 7000
-	-1   0    0    1
+P 4900 7000
+F 0 "LD10" H 5150 6850 50  0000 C CNN
+F 1 "Yellow" H 5100 7150 50  0000 C CNN
+F 2 "footprints:LED_0603" H 4900 7000 50  0001 C CNN
+F 3 "~" H 4900 7000 50  0001 C CNN
+	1    4900 7000
+	1    0    0    -1
 $EndComp
 $Comp
@@
 Wire Wire Line
 	4800 6850 4800 7000
-Wire Wire Line
-	4800 7000 5000 7000
-Wire Wire Line
-	5300 7000 5600 7000
 Wire Wire Line
 	6300 5200 6450 5200
@@
 	1    0    0    -1
 $EndComp
+Wire Wire Line
+	5450 7000 5600 7000
+Wire Wire Line
+	4800 7000 4900 7000
 $EndSCHEMATC
