File: FPGA_Lattice_Replica_Icezum/power_supply.sch (KiCad schematic (older format))
At the start: 53 parts, among them J18 Power_Jack, Q1 DMP3017, Q2 DMP3017, Q3 DMP2035U-7, Q4 Mosfet_P_DFN-6, Q5 PMBT3906, SW3 SPDT_Switch, SW4 Switch, U10 AP7361, U11 TLV711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

Commit message: se completo esquema de perifericos y sockets. Se puso el mismo simbolo de referencia GND en el esquema de la fuente
Connections:
- net labels added: GND
Other:
- moved on the sheet: R33

Commit message: se ejecuto y se corrigio electrical rules check
Connections:
- net labels removed: GNDREF
- wire segments 197 -> 202
- no-connect marks 4 -> 6
Changed lines of the file:
@@
 	1    0    0    -1
 $EndComp
-$Comp
-L power:GNDREF #PWR?
-U 1 1 5CF6AE1E
-P 7800 4000
-F 0 "#PWR?" H 7800 3750 50  0001 C CNN
-F 1 "GNDREF" H 7805 3827 50  0001 C CNN
-F 2 "" H 7800 4000 50  0001 C CNN
-F 3 "" H 7800 4000 50  0001 C CNN
-	1    7800 4000
-	1    0    0    -1
-$EndComp
-Wire Wire Line
-	7800 3950 7800 4000
 Wire Wire Line
 	4800 3500 5350 3500
@@
 	4300 7200 4750 7200
 Wire Wire Line
-	4750 7200 4750 6150
+	4750 7200 4750 6850
 Connection ~ 4750 6150
 Wire Wire Line
@@
 $EndComp
 $Comp
-L icezum:+1V2 #PWR101
+L icezum:+1V2 #PWR0101
 U 1 1 5D13F0AA
 P 7250 1150
-F 0 "#PWR101" H 7250 1000 50  0001 C CNN
+F 0 "#PWR0101" H 7250 1000 50  0001 C CNN
 F 1 "+1V2" H 7265 1323 50  0000 C CNN
 F 2 "" H 7250 1150 60  0000 C CNN
@@
 $EndComp
 $Comp
-L icezum:PWR_FLAG #FLG105
+L icezum:PWR_FLAG #FLG0105
 U 1 1 5D1DB363
 P 10500 950
-F 0 "#FLG105" H 10500 1045 50  0001 C CNN
+F 0 "#FLG0105" H 10500 1045 50  0001 C CNN
 F 1 "PWR_FLAG" V 10500 1128 50  0000 L CNN
 F 2 "" H 10500 950 50  0000 C CNN
@@
 	5150 7350 4900 7350
 $Comp
-L power:GND #PWR?
+L power:GND #PWR0105
 U 1 1 5D3D6D41
 P 8750 5150
-F 0 "#PWR?" H 8750 4900 50  0001 C CNN
+F 0 "#PWR0105" H 8750 4900 50  0001 C CNN
 F 1 "GND" H 8755 4977 50  0000 C CNN
 F 2 "" H 8750 5150 50  0001 C CNN
@@
 $EndComp
 $Comp
-L power:GND #PWR?
+L power:GND #PWR0106
 U 1 1 5D3D6E13
 P 8200 5150
-F 0 "#PWR?" H 8200 4900 50  0001 C CNN
+F 0 "#PWR0106" H 8200 4900 50  0001 C CNN
 F 1 "GND" H 8205 4977 50  0000 C CNN
 F 2 "" H 8200 5150 50  0001 C CNN
@@
 	8200 4750 8200 5150
 $Comp
-L power:GND #PWR?
+L power:GND #PWR0107
 U 1 1 5D3EC43A
 P 10200 4200
-F 0 "#PWR?" H 10200 3950 50  0001 C CNN
+F 0 "#PWR0107" H 10200 3950 50  0001 C CNN
 F 1 "GND" H 10200 4050 50  0000 C CNN
 F 2 "" H 10200 4200 50  0001 C CNN
@@
 $EndComp
 $Comp
-L power:GND #PWR?
+L power:GND #PWR0109
 U 1 1 5D3EC971
 P 8200 6300
-F 0 "#PWR?" H 8200 6050 50  0001 C CNN
+F 0 "#PWR0109" H 8200 6050 50  0001 C CNN
 F 1 "GND" H 8205 6127 50  0000 C CNN
 F 2 "" H 8200 6300 50  0001 C CNN
@@
 	10200 4200 10450 4200
 $Comp
-L power:GND #PWR?
+L power:GND #PWR0110
 U 1 1 5D402940
 P 4550 4550
-F 0 "#PWR?" H 4550 4300 50  0001 C CNN
+F 0 "#PWR0110" H 4550 4300 50  0001 C CNN
 F 1 "GND" H 4550 4400 50  0000 C CNN
 F 2 "" H 4550 4550 50  0001 C CNN
@@
 $EndComp
 $Comp
-L power:GND #PWR?
+L power:GND #PWR0111
 U 1 1 5D402F92
 P 3800 4550
-F 0 "#PWR?" H 3800 4300 50  0001 C CNN
+F 0 "#PWR0111" H 3800 4300 50  0001 C CNN
 F 1 "GND" H 3800 4400 50  0000 C CNN
 F 2 "" H 3800 4550 50  0001 C CNN
@@
 $EndComp
 $Comp
-L power:GND #PWR?
+L power:GND #PWR0112
 U 1 1 5D40340D
 P 3350 4550
-F 0 "#PWR?" H 3350 4300 50  0001 C CNN
+F 0 "#PWR0112" H 3350 4300 50  0001 C CNN
 F 1 "GND" H 3350 4400 50  0000 C CNN
 F 2 "" H 3350 4550 50  0001 C CNN
@@
 $EndComp
 $Comp
-L power:GND #PWR?
+L power:GND #PWR0113
 U 1 1 5D4035CF
 P 800 4950
-F 0 "#PWR?" H 800 4700 50  0001 C CNN
+F 0 "#PWR0113" H 800 4700 50  0001 C CNN
 F 1 "GND" H 800 4800 50  0000 C CNN
 F 2 "" H 800 4950 50  0001 C CNN
@@
 	800  4450 800  4950
 $Comp
-L power:GND #PWR?
+L power:GND #PWR0114
 U 1 1 5D42E72C
 P 600 6550
-F 0 "#PWR?" H 600 6300 50  0001 C CNN
+F 0 "#PWR0114" H 600 6300 50  0001 C CNN
 F 1 "GND" H 600 6400 50  0000 C CNN
 F 2 "" H 600 6550 50  0001 C CNN
@@
 $EndComp
 $Comp
-L power:GND #PWR?
+L power:GND #PWR0115
 U 1 1 5D42EAC7
 P 1500 6550
-F 0 "#PWR?" H 1500 6300 50  0001 C CNN
+F 0 "#PWR0115" H 1500 6300 50  0001 C CNN
 F 1 "GND" H 1500 6400 50  0000 C CNN
 F 2 "" H 1500 6550 50  0001 C CNN
@@
 $EndComp
 $Comp
-L power:GND #PWR?
+L power:GND #PWR0116
 U 1 1 5D42ED72
 P 1650 6900
-F 0 "#PWR?" H 1650 6650 50  0001 C CNN
+F 0 "#PWR0116" H 1650 6650 50  0001 C CNN
 F 1 "GND" H 1650 6750 50  0000 C CNN
 F 2 "" H 1650 6900 50  0001 C CNN
@@
 $EndComp
 $Comp
-L power:GND #PWR?
+L power:GND #PWR0117
 U 1 1 5D42EF7E
 P 1850 7300
-F 0 "#PWR?" H 1850 7050 50  0001 C CNN
+F 0 "#PWR0117" H 1850 7050 50  0001 C CNN
 F 1 "GND" H 1850 7150 50  0000 C CNN
 F 2 "" H 1850 7300 50  0001 C CNN
@@
 $EndComp
 $Comp
-L power:GND #PWR?
+L power:GND #PWR0118
 U 1 1 5D42F1C2
 P 2550 7600
-F 0 "#PWR?" H 2550 7350 50  0001 C CNN
+F 0 "#PWR0118" H 2550 7350 50  0001 C CNN
 F 1 "GND" H 2550 7450 50  0000 C CNN
 F 2 "" H 2550 7600 50  0001 C CNN
@@
 $EndComp
 $Comp
-L power:GND #PWR?
+L power:GND #PWR0119
 U 1 1 5D42F4B8
 P 3000 7600
-F 0 "#PWR?" H 3000 7350 50  0001 C CNN
+F 0 "#PWR0119" H 3000 7350 50  0001 C CNN
 F 1 "GND" H 3000 7450 50  0000 C CNN
 F 2 "" H 3000 7600 50  0001 C CNN
@@
 	1850 7200 1850 7300
 $Comp
-L power:GND #PWR?
+L power:GND #PWR0120
 U 1 1 5D45B596
 P 4100 6600
-F 0 "#PWR?" H 4100 6350 50  0001 C CNN
+F 0 "#PWR0120" H 4100 6350 50  0001 C CNN
 F 1 "GND" H 4100 6450 50  0000 C CNN
 F 2 "" H 4100 6600 50  0001 C CNN
@@
 $EndComp
 $Comp
-L power:GND #PWR?
+L power:GND #PWR0121
 U 1 1 5D45BAA0
 P 4500 6600
-F 0 "#PWR?" H 4500 6350 50  0001 C CNN
+F 0 "#PWR0121" H 4500 6350 50  0001 C CNN
 F 1 "GND" H 4500 6450 50  0000 C CNN
 F 2 "" H 4500 6600 50  0001 C CNN
@@
 	4500 6500 4500 6600
 $Comp
-L power:GND #PWR?
+L power:GND #PWR0122
 U 1 1 5D4717F7
 P 5950 2100
-F 0 "#PWR?" H 5950 1850 50  0001 C CNN
+F 0 "#PWR0122" H 5950 1850 50  0001 C CNN
 F 1 "GND" H 5950 1950 50  0000 C CNN
 F 2 "" H 5950 2100 50  0001 C CNN
@@
 $EndComp
 $Comp
-L power:GND #PWR?
+L power:GND #PWR0123
 U 1 1 5D471B9A
 P 1750 2400
-F 0 "#PWR?" H 1750 2150 50  0001 C CNN
+F 0 "#PWR0123" H 1750 2150 50  0001 C CNN
 F 1 "GND" H 1750 2250 50  0000 C CNN
 F 2 "" H 1750 2400 50  0001 C CNN
@@
 $EndComp
 $Comp
-L power:GND #PWR?
+L power:GND #PWR0124
 U 1 1 5D471EB5
 P 2950 2100
-F 0 "#PWR?" H 2950 1850 50  0001 C CNN
+F 0 "#PWR0124" H 2950 1850 50  0001 C CNN
 F 1 "GND" H 2950 1950 50  0000 C CNN
 F 2 "" H 2950 2100 50  0001 C CNN
@@
 	5950 2000 5950 2100
 Connection ~ 5950 2000
+Text Label 5850 7750 0    50   ~ 0
+5V_P_CTL
+Wire Wire Line
+	4900 7750 5850 7750
+Connection ~ 4900 7750
+$Comp
+L power:GND #PWR0103
+U 1 1 5D00806E
+P 7800 4050
+F 0 "#PWR0103" H 7800 3800 50  0001 C CNN
+F 1 "GND" H 7805 3877 50  0000 C CNN
+F 2 "" H 7800 4050 50  0001 C CNN
+F 3 "" H 7800 4050 50  0001 C CNN
+	1    7800 4050
+	1    0    0    -1
+$EndComp
+Wire Wire Line
+	7800 3950 7800 4050
+NoConn ~ 7700 5000
+$Comp
+L power:GND #PWR0233
+U 1 1 5D02A260
+P 7700 5250
+F 0 "#PWR0233" H 7700 5000 50  0001 C CNN
+F 1 "GND" H 7705 5077 50  0000 C CNN
+F 2 "" H 7700 5250 50  0001 C CNN
+F 3 "" H 7700 5250 50  0001 C CNN
+	1    7700 5250
+	1    0    0    -1
+$EndComp
+Wire Wire Line
+	4750 6850 3500 6850
+Wire Wire Line
+	3500 6850 3500 6600
+Wire Wire Line
+	3500 6600 3200 6600
+Connection ~ 4750 6850
+Wire Wire Line
+	4750 6850 4750 6150
+NoConn ~ 3200 5800
 $EndSCHEMATC

Commit message: se comenzo asignacion de footprints
Parts:
- C60, C62, C64, C65, C66, C70, C71: footprint (none) -> footprints:C_0603
- C67, C69: footprint (none) -> footprints:C_1206
- D10: footprint (none) -> footprints:DO-214AC
- D11: footprint (none) -> footprints:SOT-23
- D12, D2, D4: footprint (none) -> footprints:LED_0603
Changed lines of the file:
@@
 F 0 "Q1" V 3702 3850 60  0000 C CNN
 F 1 "DMP3017" V 3808 3850 60  0000 C CNN
-F 2 "" H 4540 3830 60  0000 C CNN
+F 2 "" H 4540 3830 60  0001 C CNN
 F 3 "" H 4540 3830 60  0000 C CNN
 	1    4100 3500
@@
 F 0 "Q2" V 6102 3850 60  0000 C CNN
 F 1 "DMP3017" V 6208 3850 60  0000 C CNN
-F 2 "" H 6940 3830 60  0000 C CNN
+F 2 "" H 6940 3830 60  0001 C CNN
 F 3 "" H 6940 3830 60  0000 C CNN
 	1    6500 3500
@@
 F 0 "Q3" V 7502 3975 60  0000 C CNN
 F 1 "DMP2035U-7" V 7608 3975 60  0000 C CNN
-F 2 "" H 8350 3950 60  0000 C CNN
+F 2 "" H 8350 3950 60  0001 C CNN
 F 3 "" H 8350 3950 60  0000 C CNN
 	1    8350 3950
@@
 F 0 "D10" H 3850 3550 60  0000 L CNN
 F 1 "SMAJ17CA" V 3600 3150 60  0000 L CNN
-F 2 "" H 3800 3710 60  0000 C CNN
+F 2 "footprints:DO-214AC" H 3800 3710 60  0001 C CNN
 F 3 "" H 3800 3710 60  0000 C CNN
 	1    3800 3650
@@
 F 0 "C62" V 5398 3950 50  0000 C CNN
 F 1 "100 nF" V 5489 3950 50  0000 C CNN
-F 2 "" H 5688 3800 50  0001 C CNN
+F 2 "footprints:C_0603" H 5688 3800 50  0001 C CNN
 F 3 "~" H 5650 3950 50  0001 C CNN
 	1    5650 3950
@@
 F 0 "D2" V 9200 4950 60  0000 R CNN
 F 1 "BZX384C5V1-E3" H 9250 5150 60  0000 R CNN
-F 2 "" H 8750 5000 60  0000 C CNN
+F 2 "footprints:LED_0603" H 8750 5000 60  0001 C CNN
 F 3 "" H 8750 5000 60  0000 C CNN
 	1    8750 5000
@@
 F 0 "TP6" H 6778 3442 60  0000 L CNN
 F 1 "TestPoint_Small" H 6700 3250 60  0001 C CNN
-F 2 "" H 6700 3350 60  0000 C CNN
+F 2 "" H 6700 3350 60  0001 C CNN
 F 3 "" H 6700 3350 60  0000 C CNN
 	1    6700 3350
@@
 F 0 "D11" H 6525 5269 60  0000 C CNN
 F 1 "BAT54C-G3-08" H 6525 5163 60  0000 C CNN
-F 2 "" H 6200 5000 60  0000 C CNN
+F 2 "footprints:SOT-23" H 6200 5000 60  0001 C CNN
 F 3 "" H 6200 5000 60  0000 C CNN
 	1    6200 5000
@@
 F 0 "SW3" H 7325 5441 47  0000 C CNN
 F 1 "SPDT_Switch" H 7325 5354 47  0000 C CNN
-F 2 "" H 6950 5100 60  0000 C CNN
+F 2 "" H 6950 5100 60  0001 C CNN
 F 3 "" H 6950 5100 60  0000 C CNN
 	1    6950 5100
@@
 F 0 "C60" H 6700 3850 50  0000 L CNN
 F 1 "10 nF" H 6700 3650 50  0000 L CNN
-F 2 "" H 6738 3600 50  0001 C CNN
+F 2 "footprints:C_0603" H 6738 3600 50  0001 C CNN
 F 3 "~" H 6700 3750 50  0001 C CNN
 	1    6700 3750
@@
 F 0 "TP7" H 7878 3386 60  0000 L CNN
 F 1 "TestPoint_Small" H 7800 3250 60  0001 C CNN
-F 2 "" H 7800 3350 60  0000 C CNN
+F 2 "" H 7800 3350 60  0001 C CNN
 F 3 "" H 7800 3350 60  0000 C CNN
 	1    7800 3350
@@
 F 0 "U12" H 2650 6099 60  0000 C CNN
 F 1 "TPS62133RGTR" H 2650 5993 60  0000 C CNN
-F 2 "" H 2210 5910 60  0000 C CNN
+F 2 "" H 2210 5910 60  0001 C CNN
 F 3 "" H 2210 5910 60  0000 C CNN
 	1    2100 5800
@@
 F 0 "L4" H 1075 6244 60  0000 C CNN
 F 1 "Ferrite_Bead" H 780 5890 60  0001 L BNN
-F 2 "" H 750 6000 60  0000 C CNN
+F 2 "" H 750 6000 60  0001 C CNN
 F 3 "" H 750 6000 60  0000 C CNN
 F 4 "BLM18SG121TN1D" H 1075 6138 60  0000 C CNN "OrderingCode"
@@
 F 0 "C66" H 715 6346 50  0000 L CNN
 F 1 "100 nF" H 715 6255 50  0000 L CNN
-F 2 "" H 638 6150 50  0001 C CNN
+F 2 "footprints:C_0603" H 638 6150 50  0001 C CNN
 F 3 "~" H 600 6300 50  0001 C CNN
 	1    600  6300
@@
 F 0 "C67" H 1615 6346 50  0000 L CNN
 F 1 "10 uF" H 1615 6255 50  0000 L CNN
-F 2 "" H 1538 6150 50  0001 C CNN
+F 2 "footprints:C_1206" H 1538 6150 50  0001 C CNN
 F 3 "~" H 1500 6300 50  0001 C CNN
 	1    1500 6300
@@
 F 0 "C70" H 1765 6696 50  0000 L CNN
 F 1 "100 nF" H 1765 6605 50  0000 L CNN
-F 2 "" H 1688 6500 50  0001 C CNN
+F 2 "footprints:C_0603" H 1688 6500 50  0001 C CNN
 F 3 "~" H 1650 6650 50  0001 C CNN
 	1    1650 6650
@@
 F 0 "C71" H 1965 7096 50  0000 L CNN
 F 1 "620 nF" H 1965 7005 50  0000 L CNN
-F 2 "" H 1888 6900 50  0001 C CNN
+F 2 "footprints:C_0603" H 1888 6900 50  0001 C CNN
 F 3 "~" H 1850 7050 50  0001 C CNN
 	1    1850 7050
@@
 F 0 "L5" H 3750 6394 60  0000 C CNN
 F 1 "2.2 uH 4,7A" H 3750 6288 60  0000 C CNN
-F 2 "" H 3400 6150 60  0000 C CNN
+F 2 "" H 3400 6150 60  0001 C CNN
 F 3 "" H 3400 6150 60  0000 C CNN
 	1    3400 6150
@@
 F 0 "TP5" H 6878 5892 60  0000 L CNN
 F 1 "TestPoint_Small" H 6800 5700 60  0001 C CNN
-F 2 "" H 6800 5800 60  0000 C CNN
+F 2 "" H 6800 5800 60  0001 C CNN
 F 3 "" H 6800 5800 60  0000 C CNN
 	1    6800 5800
@@
 F 0 "TP1" H 4828 5892 60  0000 L CNN
 F 1 "TestPoint_Small" H 4750 5700 60  0001 C CNN
-F 2 "" H 4750 5800 60  0000 C CNN
+F 2 "" H 4750 5800 60  0001 C CNN
 F 3 "" H 4750 5800 60  0000 C CNN
 	1    4750 5800
@@
 F 0 "Q4" V 5752 6500 60  0000 C CNN
 F 1 "Mosfet_P_DFN-6" V 5858 6500 60  0000 C CNN
-F 2 "" H 6590 6480 60  0000 C CNN
+F 2 "" H 6590 6480 60  0001 C CNN
 F 3 "" H 6590 6480 60  0000 C CNN
 	1    6150 6150
@@
 F 0 "C69" H 4550 6450 50  0000 L CNN
 F 1 "22 uF" H 4500 6250 50  0000 L CNN
-F 2 "" H 4538 6200 50  0001 C CNN
+F 2 "footprints:C_1206" H 4538 6200 50  0001 C CNN
 F 3 "~" H 4500 6350 50  0001 C CNN
 	1    4500 6350
@@
 F 0 "SW4" H 9000 6250 60  0000 C CNN
 F 1 "Switch" H 9000 5950 60  0000 C CNN
-F 2 "" H 8600 6050 60  0000 C CNN
+F 2 "" H 8600 6050 60  0001 C CNN
 F 3 "" H 8600 6050 60  0000 C CNN
 	1    8600 6050
@@
 F 0 "D4" H 9850 6450 50  0000 C CNN
 F 1 "NSR0530HT1G" H 9850 6250 50  0000 C CNN
-F 2 "" H 9850 6350 50  0000 C CNN
+F 2 "footprints:LED_0603" H 9850 6350 50  0001 C CNN
 F 3 "" H 9850 6350 50  0000 C CNN
 	1    9850 6350
@@
 F 0 "D12" V 839 4182 50  0000 R CNN
 F 1 "WHITE" V 748 4182 50  0000 R CNN
-F 2 "" H 800 4300 50  0001 C CNN
+F 2 "footprints:LED_0603" H 800 4300 50  0001 C CNN
 F 3 "~" H 800 4300 50  0001 C CNN
 	1    800  4300
@@
 F 0 "U10" H 3100 1899 60  0000 C CNN
 F 1 "AP7361" H 3100 1793 60  0000 C CNN
-F 2 "" H 2670 1710 60  0000 C CNN
+F 2 "" H 2670 1710 60  0001 C CNN
 F 3 "" H 2670 1710 60  0000 C CNN
 	1    2450 1600
@@
 F 0 "TP2" H 3428 1242 60  0000 L CNN
 F 1 "TestPoint_Small" H 3350 1050 60  0001 C CNN
-F 2 "" H 3350 1150 60  0000 C CNN
+F 2 "" H 3350 1150 60  0001 C CNN
 F 3 "" H 3350 1150 60  0000 C CNN
 	1    3350 1150
@@
 F 0 "TP3" H 7528 1642 60  0000 L CNN
 F 1 "TestPoint_Small" H 7450 1450 60  0001 C CNN
-F 2 "" H 7450 1550 60  0000 C CNN
+F 2 "" H 7450 1550 60  0001 C CNN
 F 3 "" H 7450 1550 60  0000 C CNN
 	1    7450 1550
@@
 F 0 "TP4" H 6828 1642 60  0000 L CNN
 F 1 "TestPoint_Small" H 6750 1450 60  0001 C CNN
-F 2 "" H 6750 1550 60  0000 C CNN
+F 2 "" H 6750 1550 60  0001 C CNN
 F 3 "" H 6750 1550 60  0000 C CNN
 	1    6750 1550
@@
 F 0 "C64" H 7365 1896 50  0000 L CNN
 F 1 "4.7 uF" H 7365 1805 50  0000 L CNN
-F 2 "" H 7288 1700 50  0001 C CNN
+F 2 "footprints:C_0603" H 7288 1700 50  0001 C CNN
 F 3 "~" H 7250 1850 50  0001 C CNN
 	1    7250 1850
@@
 F 0 "C65" H 6615 1896 50  0000 L CNN
 F 1 "4.7 uF" H 6615 1805 50  0000 L CNN
-F 2 "" H 6538 1700 50  0001 C CNN
+F 2 "footprints:C_0603" H 6538 1700 50  0001 C CNN
 F 3 "~" H 6500 1850 50  0001 C CNN
 	1    6500 1850
@@
 F 0 "U11" H 5350 1899 60  0000 C CNN
 F 1 "TLV711" H 5350 1793 60  0000 C CNN
-F 2 "" H 4970 1710 60  0000 C CNN
+F 2 "" H 4970 1710 60  0001 C CNN
 F 3 "" H 4970 1710 60  0000 C CNN
 	1    4750 1600
