File: FPGA_Lattice_Replica_Icezum/power_supply.sch (KiCad schematic (older format))
At the start: 53 parts, among them J18 Power_Jack, Q1 DMP3017, Q2 DMP3017, Q3 DMP2035U-7, Q4 Mosfet_P_DFN-6, Q5 PMBT3906, SW3 SPDT_Switch, SW4 Switch, U10 AP7361, U11 TLV711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

Commit message: se mejoro esquematico de acuerdo a la revisión del docente. Se mejoro rotulo (se coloco link del repo, autor y autor de la versión original y la licencia) se mejoro el flujo izquiera derecha de los botones, se desplazo fiduciales a la página principal, se achico el esquematico en la parte de headers
Parts:
- C59, C60, C61, C62, C64, C65, C66, C70, C71: footprint footprints:C_0603 -> footprints:L_0805
- C63, C68: footprint footprints:C_0402 -> footprints:L_0805
- R24, R25, R26, R27, R28, R29, R30, R33, R34, R35, R36, R37, R38, R39: footprint footprints:R_0402 -> footprints:F_0805
Changed lines of the file:
@@
 encoding utf-8
 Sheet 2 6
-Title ""
+Title "Power Supply"
 Date "2019-06-03"
 Rev "v1.0"
 Comp "Especialización en Sistemas Embebidos - DCI (7 Cohorte )"
 Comment1 "Proyecto para trabajo final de la materia DCI - CESE-7Co2018"
-Comment2 "Revisor del trabajo: Gustavo Paredes Delayone"
-Comment3 "Revisor suplente : Rafael Oliva curso CESE en la 6 Cohorte"
-Comment4 ""
+Comment2 "Revisores del trabajo: Gustavo Paredes Delayone, Rafael Oliva curso CESE en la 6 Cohorte"
+Comment3 "License: Creative commons Attribution ShareAlike"
+Comment4 "Autor: Jacobo O. Salvador. Adaptador versión  original (Eladio Delgado Mingorance)"
 $EndDescr
 $Comp
@@
 F 0 "C61" V 5302 3950 50  0000 C CNN
 F 1 "10 nF" V 5211 3950 50  0000 C CNN
-F 2 "footprints:C_0603" H 5088 3800 50  0001 C CNN
+F 2 "footprints:L_0805" H 5088 3800 50  0001 C CNN
 F 3 "~" H 5050 3950 50  0001 C CNN
 F 4 "X7R" V 5050 3950 50  0001 C CNN "Clase"
@@
 F 0 "C62" V 5398 3950 50  0000 C CNN
 F 1 "100 nF" V 5489 3950 50  0000 C CNN
-F 2 "footprints:C_0603" H 5688 3800 50  0001 C CNN
+F 2 "footprints:L_0805" H 5688 3800 50  0001 C CNN
 F 3 "~" H 5650 3950 50  0001 C CNN
 	1    5650 3950
@@
 F 0 "R25" H 4620 4296 50  0000 L CNN
 F 1 "10K±5% 0.063 W" V 4450 3900 50  0000 L CNN
-F 2 "footprints:R_0402" V 4480 4250 50  0001 C CNN
+F 2 "footprints:F_0805" V 4480 4250 50  0001 C CNN
 F 3 "~" H 4550 4250 50  0001 C CNN
 	1    4550 4250
@@
 F 0 "R26" H 5420 4296 50  0000 L CNN
 F 1 "100K±5% 0.063 W" V 5250 3800 50  0000 L CNN
-F 2 "footprints:R_0402" V 5280 4250 50  0001 C CNN
+F 2 "footprints:F_0805" V 5280 4250 50  0001 C CNN
 F 3 "~" H 5350 4250 50  0001 C CNN
 	1    5350 4250
@@
 F 0 "R27" H 6120 4296 50  0000 L CNN
 F 1 "10K±5% 0.063 W" V 5950 3800 50  0000 L CNN
-F 2 "footprints:R_0402" V 5980 4250 50  0001 C CNN
+F 2 "footprints:F_0805" V 5980 4250 50  0001 C CNN
 F 3 "~" H 6050 4250 50  0001 C CNN
 	1    6050 4250
@@
 F 0 "R29" H 8270 4646 50  0000 L CNN
 F 1 "100K±5% 0.063 W" V 8100 4000 50  0000 L CNN
-F 2 "footprints:R_0402" V 8130 4600 50  0001 C CNN
+F 2 "footprints:F_0805" V 8130 4600 50  0001 C CNN
 F 3 "~" H 8200 4600 50  0001 C CNN
 	1    8200 4600
@@
 F 0 "R28" V 7593 4450 50  0000 C CNN
 F 1 "10K±5% 0.063 W" V 7684 4450 50  0000 C CNN
-F 2 "footprints:R_0402" V 7730 4450 50  0001 C CNN
+F 2 "footprints:F_0805" V 7730 4450 50  0001 C CNN
 F 3 "~" H 7800 4450 50  0001 C CNN
 	1    7800 4450
@@
 F 0 "R38" V 7150 3750 50  0000 C CNN
 F 1 "10K±5% 0.063 W" V 7350 3800 50  0000 C CNN
-F 2 "footprints:R_0402" V 7180 3750 50  0001 C CNN
+F 2 "footprints:F_0805" V 7180 3750 50  0001 C CNN
 F 3 "~" H 7250 3750 50  0001 C CNN
 	1    7250 3750
@@
 F 0 "R39" H 7870 3846 50  0000 L CNN
 F 1 "1K±5% 0.063 W" V 7700 3450 50  0000 L CNN
-F 2 "footprints:R_0402" V 7730 3800 50  0001 C CNN
+F 2 "footprints:F_0805" V 7730 3800 50  0001 C CNN
 F 3 "~" H 7800 3800 50  0001 C CNN
 	1    7800 3800
@@
 F 0 "C60" H 6700 3850 50  0000 L CNN
 F 1 "10 nF" H 6700 3650 50  0000 L CNN
-F 2 "footprints:C_0603" H 6738 3600 50  0001 C CNN
+F 2 "footprints:L_0805" H 6738 3600 50  0001 C CNN
 F 3 "~" H 6700 3750 50  0001 C CNN
 	1    6700 3750
@@
 F 0 "R24" V 6300 3950 50  0000 C CNN
 F 1 "10K±5% 0.063 W" V 6500 3950 50  0000 C CNN
-F 2 "footprints:R_0402" V 6330 3950 50  0001 C CNN
+F 2 "footprints:F_0805" V 6330 3950 50  0001 C CNN
 F 3 "~" H 6400 3950 50  0001 C CNN
 	1    6400 3950
@@
 F 0 "C66" H 715 6346 50  0000 L CNN
 F 1 "100 nF" H 715 6255 50  0000 L CNN
-F 2 "footprints:C_0603" H 638 6150 50  0001 C CNN
+F 2 "footprints:L_0805" H 638 6150 50  0001 C CNN
 F 3 "~" H 600 6300 50  0001 C CNN
 	1    600  6300
@@
 F 0 "C70" H 1765 6696 50  0000 L CNN
 F 1 "100 nF" H 1765 6605 50  0000 L CNN
-F 2 "footprints:C_0603" H 1688 6500 50  0001 C CNN
+F 2 "footprints:L_0805" H 1688 6500 50  0001 C CNN
 F 3 "~" H 1650 6650 50  0001 C CNN
 	1    1650 6650
@@
 F 0 "C71" H 1965 7096 50  0000 L CNN
 F 1 "620 nF" H 1965 7005 50  0000 L CNN
-F 2 "footprints:C_0603" H 1888 6900 50  0001 C CNN
+F 2 "footprints:L_0805" H 1888 6900 50  0001 C CNN
 F 3 "~" H 1850 7050 50  0001 C CNN
 	1    1850 7050
@@
 F 0 "C68" H 4150 6450 50  0000 L CNN
 F 1 "100 nF" H 4150 6250 50  0000 L CNN
-F 2 "footprints:C_0402" H 4138 6200 50  0001 C CNN
+F 2 "footprints:L_0805" H 4138 6200 50  0001 C CNN
 F 3 "~" H 4100 6350 50  0001 C CNN
 	1    4100 6350
@@
 F 0 "C63" H 6565 6746 50  0000 L CNN
 F 1 "100 nF" H 6565 6655 50  0000 L CNN
-F 2 "footprints:C_0402" H 6488 6550 50  0001 C CNN
+F 2 "footprints:L_0805" H 6488 6550 50  0001 C CNN
 F 3 "~" H 6450 6700 50  0001 C CNN
 	1    6450 6700
@@
 F 0 "R33" V 5100 7400 50  0000 C CNN
 F 1 "10K±5% 0.063 W" V 5200 7400 50  0000 C CNN
-F 2 "footprints:R_0402" V 5230 7350 50  0001 C CNN
+F 2 "footprints:F_0805" V 5230 7350 50  0001 C CNN
 F 3 "~" H 5300 7350 50  0001 C CNN
 	1    5300 7350
@@
 F 0 "R35" V 5900 7350 50  0000 C CNN
 F 1 "100K±5% 0.063 W" V 6000 7300 50  0000 C CNN
-F 2 "footprints:R_0402" V 6030 7350 50  0001 C CNN
+F 2 "footprints:F_0805" V 6030 7350 50  0001 C CNN
 F 3 "~" H 6100 7350 50  0001 C CNN
 	1    6100 7350
@@
 F 0 "R36" H 4900 6700 50  0000 L CNN
 F 1 "100K±5% 0.063 W" V 5100 6200 50  0000 L CNN
-F 2 "footprints:R_0402" V 4830 6550 50  0001 C CNN
+F 2 "footprints:F_0805" V 4830 6550 50  0001 C CNN
 F 3 "~" H 4900 6550 50  0001 C CNN
 	1    4900 6550
@@
 F 0 "R37" H 4970 7646 50  0000 L CNN
 F 1 "10K±5% 0.063 W" H 4970 7555 50  0000 L CNN
-F 2 "footprints:R_0402" V 4830 7600 50  0001 C CNN
+F 2 "footprints:F_0805" V 4830 7600 50  0001 C CNN
 F 3 "~" H 4900 7600 50  0001 C CNN
 	1    4900 7600
@@
 F 0 "R30" H 9520 5396 50  0000 L CNN
 F 1 "10K±5% 0.063 W" V 9350 5000 50  0000 L CNN
-F 2 "footprints:R_0402" V 9380 5350 50  0001 C CNN
+F 2 "footprints:F_0805" V 9380 5350 50  0001 C CNN
 F 3 "~" H 9450 5350 50  0001 C CNN
 	1    9450 5350
@@
 F 0 "R34" H 870 3696 50  0000 L CNN
 F 1 "10K±5% 0.063 W" H 870 3605 50  0000 L CNN
-F 2 "footprints:R_0402" V 730 3650 50  0001 C CNN
+F 2 "footprints:F_0805" V 730 3650 50  0001 C CNN
 F 3 "~" H 800 3650 50  0001 C CNN
 	1    800  3650
@@
 F 0 "C59" H 3065 1796 50  0000 L CNN
 F 1 "4.7 uF" H 3065 1705 50  0000 L CNN
-F 2 "footprints:C_0603" H 2988 1600 50  0001 C CNN
+F 2 "footprints:L_0805" H 2988 1600 50  0001 C CNN
 F 3 "~" H 2950 1750 50  0001 C CNN
 	1    2950 1750
@@
 F 0 "C64" H 7365 1896 50  0000 L CNN
 F 1 "4.7 uF" H 7365 1805 50  0000 L CNN
-F 2 "footprints:C_0603" H 7288 1700 50  0001 C CNN
+F 2 "footprints:L_0805" H 7288 1700 50  0001 C CNN
 F 3 "~" H 7250 1850 50  0001 C CNN
 	1    7250 1850
@@
 F 0 "C65" H 6615 1896 50  0000 L CNN
 F 1 "4.7 uF" H 6615 1805 50  0000 L CNN
-F 2 "footprints:C_0603" H 6538 1700 50  0001 C CNN
+F 2 "footprints:L_0805" H 6538 1700 50  0001 C CNN
 F 3 "~" H 6500 1850 50  0001 C CNN
 	1    6500 1850
