File: FPGA_Lattice_Replica_Icezum/Peripherical.sch (KiCad schematic (older format))
At the start: 33 parts, among them J15 1x4_male_pin_Header_2.54mm, J16 1x4_male_pin_Header_2.54mm, J17 1x4_male_pin_Header_2.54mm, SW1 SW1, SW2 Switch_4p, U7 ADS7924

Commit message: se ejecuto y se corrigio electrical rules check
Parts:
- gave numbers to parts that had none: 1
Connections:
- net +5V: now also JP1.3
Changed lines of the file:
@@
 $EndComp
 $Comp
-L power:GND #PWR?
+L power:GND #PWR0178
 U 1 1 5D1D7A96
 P 9650 5700
-F 0 "#PWR?" H 9650 5450 50  0001 C CNN
+F 0 "#PWR0178" H 9650 5450 50  0001 C CNN
 F 1 "GND" H 9655 5527 50  0000 C CNN
 F 2 "" H 9650 5700 50  0001 C CNN
@@
 $EndComp
 $Comp
-L icezum:Jumper_3pin JP?
+L icezum:Jumper_3pin JP1
 U 1 1 5D1EF29F
 P 1850 1000
-F 0 "JP?" V 1753 915 60  0000 R CNN
+F 0 "JP1" V 1753 915 60  0000 R CNN
 F 1 "Jumper_3pin" V 1647 915 60  0000 R CNN
 F 2 "" H 1750 1000 60  0000 C CNN
@@
 $EndComp
 $Comp
-L icezum:+3V3 #PWR?
+L icezum:+3V3 #PWR0179
 U 1 1 5D1EFD75
 P 4650 1650
-F 0 "#PWR?" H 4650 1500 50  0001 C CNN
+F 0 "#PWR0179" H 4650 1500 50  0001 C CNN
 F 1 "+3V3" H 4665 1823 50  0000 C CNN
 F 2 "" H 4650 1650 60  0000 C CNN
@@
 $EndComp
 $Comp
-L icezum:+5V #PWR?
+L icezum:+5V #PWR0180
 U 1 1 5D1F0332
 P 1650 800
-F 0 "#PWR?" H 1650 650 50  0001 C CNN
+F 0 "#PWR0180" H 1650 650 50  0001 C CNN
 F 1 "+5V" H 1665 973 50  0000 C CNN
 F 2 "" H 1650 800 60  0000 C CNN
@@
 $EndComp
 $Comp
-L power:GND #PWR?
+L power:GND #PWR0181
 U 1 1 5D1F0D21
 P 4700 4050
-F 0 "#PWR?" H 4700 3800 50  0001 C CNN
+F 0 "#PWR0181" H 4700 3800 50  0001 C CNN
 F 1 "GND" H 4705 3877 50  0000 C CNN
 F 2 "" H 4700 4050 50  0001 C CNN
@@
 Connection ~ 4950 1900
 $Comp
-L power:GND #PWR?
+L power:GND #PWR0182
 U 1 1 5D1F9CEA
 P 3700 2100
-F 0 "#PWR?" H 3700 1850 50  0001 C CNN
+F 0 "#PWR0182" H 3700 1850 50  0001 C CNN
 F 1 "GND" H 3705 1927 50  0000 C CNN
 F 2 "" H 3700 2100 50  0001 C CNN
@@
 	2450 3650 2900 3650
 $Comp
-L icezum:+5V_P #PWR?
+L icezum:+5V_P #PWR0183
 U 1 1 5D20BD3C
 P 1950 3050
-F 0 "#PWR?" H 1950 2900 50  0001 C CNN
+F 0 "#PWR0183" H 1950 2900 50  0001 C CNN
 F 1 "+5V_P" H 1965 3223 50  0000 C CNN
 F 2 "" H 1950 3050 60  0000 C CNN
@@
 $EndComp
 $Comp
-L power:GND #PWR?
+L power:GND #PWR0184
 U 1 1 5D20C4F0
 P 1300 4050
-F 0 "#PWR?" H 1300 3800 50  0001 C CNN
+F 0 "#PWR0184" H 1300 3800 50  0001 C CNN
 F 1 "GND" H 1305 3877 50  0000 C CNN
 F 2 "" H 1300 4050 50  0001 C CNN
@@
 	2800 3150 2900 3150
 $Comp
-L power:GND #PWR?
+L power:GND #PWR0185
 U 1 1 5D224015
 P 2850 4050
-F 0 "#PWR?" H 2850 3800 50  0001 C CNN
+F 0 "#PWR0185" H 2850 3800 50  0001 C CNN
 F 1 "GND" H 2855 3877 50  0000 C CNN
 F 2 "" H 2850 4050 50  0001 C CNN
@@
 	2850 3900 2900 3900
 $Comp
-L power:GND #PWR?
+L power:GND #PWR0186
 U 1 1 5D227699
 P 3650 4300
-F 0 "#PWR?" H 3650 4050 50  0001 C CNN
+F 0 "#PWR0186" H 3650 4050 50  0001 C CNN
 F 1 "GND" H 3655 4127 50  0000 C CNN
 F 2 "" H 3650 4300 50  0001 C CNN
@@
 $EndComp
 $Comp
-L power:GND #PWR?
+L power:GND #PWR0187
 U 1 1 5D2467EA
 P 3150 7100
-F 0 "#PWR?" H 3150 6850 50  0001 C CNN
+F 0 "#PWR0187" H 3150 6850 50  0001 C CNN
 F 1 "GND" H 3155 6927 50  0000 C CNN
 F 2 "" H 3150 7100 50  0001 C CNN
@@
 $EndComp
 $Comp
-L power:GND #PWR?
+L power:GND #PWR0188
 U 1 1 5D2468EF
 P 3650 7100
-F 0 "#PWR?" H 3650 6850 50  0001 C CNN
+F 0 "#PWR0188" H 3650 6850 50  0001 C CNN
 F 1 "GND" H 3655 6927 50  0000 C CNN
 F 2 "" H 3650 7100 50  0001 C CNN
@@
 $EndComp
 $Comp
-L power:GND #PWR?
+L power:GND #PWR0189
 U 1 1 5D246AC6
 P 3650 6000
-F 0 "#PWR?" H 3650 5750 50  0001 C CNN
+F 0 "#PWR0189" H 3650 5750 50  0001 C CNN
 F 1 "GND" H 3655 5827 50  0000 C CNN
 F 2 "" H 3650 6000 50  0001 C CNN
@@
 $EndComp
 $Comp
-L power:GND #PWR?
+L power:GND #PWR0190
 U 1 1 5D246D56
 P 3150 6000
-F 0 "#PWR?" H 3150 5750 50  0001 C CNN
+F 0 "#PWR0190" H 3150 5750 50  0001 C CNN
 F 1 "GND" H 3155 5827 50  0000 C CNN
 F 2 "" H 3150 6000 50  0001 C CNN
@@
 $EndComp
 $Comp
-L icezum:+3V3 #PWR?
+L icezum:+3V3 #PWR0191
 U 1 1 5D24A862
 P 5550 5450
-F 0 "#PWR?" H 5550 5300 50  0001 C CNN
+F 0 "#PWR0191" H 5550 5300 50  0001 C CNN
 F 1 "+3V3" H 5565 5623 50  0000 C CNN
 F 2 "" H 5550 5450 60  0000 C CNN
@@
 $EndComp
 $Comp
-L icezum:+3V3 #PWR?
+L icezum:+3V3 #PWR0192
 U 1 1 5D24AE69
 P 5500 6550
-F 0 "#PWR?" H 5500 6400 50  0001 C CNN
+F 0 "#PWR0192" H 5500 6400 50  0001 C CNN
 F 1 "+3V3" H 5515 6723 50  0000 C CNN
 F 2 "" H 5500 6550 60  0000 C CNN
@@
 	3150 6650 2850 6650
 Connection ~ 3150 6650
+Wire Wire Line
+	1650 800  1650 1000
 $EndSCHEMATC

Commit message: se comenzo asignacion de footprints
Parts:
- C41: footprint (none) -> footprints:C_0603
Changed lines of the file:
@@
 F 0 "U7" H 3675 3099 60  0000 C CNN
 F 1 "ADS7924" H 3675 2993 60  0000 C CNN
-F 2 "" H 3120 2910 60  0000 C CNN
+F 2 "" H 3120 2910 60  0001 C CNN
 F 3 "" H 3120 2910 60  0000 C CNN
 	1    2900 2800
@@
 F 0 "J17" H 2343 4111 60  0000 C CNN
 F 1 "1x4_male_pin_Header_2.54mm" H 2340 3460 60  0001 C CNN
-F 2 "" H 2450 4200 60  0000 C CNN
+F 2 "" H 2450 4200 60  0001 C CNN
 F 3 "" H 2450 4200 60  0000 C CNN
 	1    2450 3650
@@
 F 0 "J15" H 1743 4111 60  0000 C CNN
 F 1 "1x4_male_pin_Header_2.54mm" H 1740 3460 60  0001 C CNN
-F 2 "" H 1850 4200 60  0000 C CNN
+F 2 "" H 1850 4200 60  0001 C CNN
 F 3 "" H 1850 4200 60  0000 C CNN
 	1    1850 3650
@@
 F 0 "J16" H 1093 4111 60  0000 C CNN
 F 1 "1x4_male_pin_Header_2.54mm" H 1090 3460 60  0001 C CNN
-F 2 "" H 1200 4200 60  0000 C CNN
+F 2 "" H 1200 4200 60  0001 C CNN
 F 3 "" H 1200 4200 60  0000 C CNN
 	1    1200 3650
@@
 F 0 "C41" V 2998 1400 50  0000 C CNN
 F 1 "4.7 uF" V 3089 1400 50  0000 C CNN
-F 2 "" H 3288 1250 50  0001 C CNN
+F 2 "footprints:C_0603" H 3288 1250 50  0001 C CNN
 F 3 "~" H 3250 1400 50  0001 C CNN
 	1    3250 1400
@@
 F 0 "JP1" V 1753 915 60  0000 R CNN
 F 1 "Jumper_3pin" V 1647 915 60  0000 R CNN
-F 2 "" H 1750 1000 60  0000 C CNN
+F 2 "" H 1750 1000 60  0001 C CNN
 F 3 "" H 1750 1000 60  0000 C CNN
 	1    1850 1000
@@
 F 0 "SW1" H 4575 5743 60  0000 C CNN
 F 1 "SW1" H 4575 5743 60  0001 C CNN
-F 2 "" H 4200 5550 60  0000 C CNN
+F 2 "" H 4200 5550 60  0001 C CNN
 F 3 "" H 4200 5550 60  0000 C CNN
 	1    4200 5550
@@
 F 0 "SW2" H 4625 6843 60  0000 C CNN
 F 1 "Switch_4p" H 4625 6843 60  0001 C CNN
-F 2 "" H 4250 6650 60  0000 C CNN
+F 2 "" H 4250 6650 60  0001 C CNN
 F 3 "" H 4250 6650 60  0000 C CNN
 	1    4250 6650

Commit message: se finalizo asignación de footprint de acuerdo al modelo original de la icezum alhambra
Parts:
- C34, C35, C45, C46: footprint (none) -> footprints:C_0402
- J15, J16, J17: footprint (none) -> footprints:1x04-pin-header-2.54mm
- JP1: footprint (none) -> footprints:1x03-pin-header-2.54mm
- LD0, LD1, LD2, LD3, LD4, LD5, LD6, LD7: footprint (none) -> footprints:LED_0603
- R17, R18: footprint (none) -> footprints:R_Array_Convex_4x0603
- R19, R20, R21, R31, R32, R40, R41, R42, R43, R44, R45: footprint (none) -> footprints:R_0402
- SW1, SW2: footprint (none) -> footprints:SW_SMD_60X3.8
- U7: footprint (none) -> footprints:QFN16
Changed lines of the file:
@@
 F 0 "LD0" H 9193 1245 50  0000 C CNN
 F 1 "Green" H 9193 1336 50  0000 C CNN
-F 2 "" H 9200 1500 50  0001 C CNN
+F 2 "footprints:LED_0603" H 9200 1500 50  0001 C CNN
 F 3 "~" H 9200 1500 50  0001 C CNN
 	1    9200 1500
@@
 F 0 "LD1" H 9193 1745 50  0000 C CNN
 F 1 "Green" H 9193 1836 50  0000 C CNN
-F 2 "" H 9200 2000 50  0001 C CNN
+F 2 "footprints:LED_0603" H 9200 2000 50  0001 C CNN
 F 3 "~" H 9200 2000 50  0001 C CNN
 	1    9200 2000
@@
 F 0 "LD2" H 9193 2295 50  0000 C CNN
 F 1 "Green" H 9193 2386 50  0000 C CNN
-F 2 "" H 9200 2550 50  0001 C CNN
+F 2 "footprints:LED_0603" H 9200 2550 50  0001 C CNN
 F 3 "~" H 9200 2550 50  0001 C CNN
 	1    9200 2550
@@
 F 0 "LD3" H 9193 2845 50  0000 C CNN
 F 1 "Green" H 9193 2936 50  0000 C CNN
-F 2 "" H 9200 3100 50  0001 C CNN
+F 2 "footprints:LED_0603" H 9200 3100 50  0001 C CNN
 F 3 "~" H 9200 3100 50  0001 C CNN
 	1    9200 3100
@@
 F 0 "LD4" H 9193 3445 50  0000 C CNN
 F 1 "Green" H 9193 3536 50  0000 C CNN
-F 2 "" H 9200 3700 50  0001 C CNN
+F 2 "footprints:LED_0603" H 9200 3700 50  0001 C CNN
 F 3 "~" H 9200 3700 50  0001 C CNN
 	1    9200 3700
@@
 F 0 "LD5" H 9193 4045 50  0000 C CNN
 F 1 "Green" H 9193 4136 50  0000 C CNN
-F 2 "" H 9200 4300 50  0001 C CNN
+F 2 "footprints:LED_0603" H 9200 4300 50  0001 C CNN
 F 3 "~" H 9200 4300 50  0001 C CNN
 	1    9200 4300
@@
 F 0 "LD6" H 9193 4595 50  0000 C CNN
 F 1 "Green" H 9193 4686 50  0000 C CNN
-F 2 "" H 9200 4850 50  0001 C CNN
+F 2 "footprints:LED_0603" H 9200 4850 50  0001 C CNN
 F 3 "~" H 9200 4850 50  0001 C CNN
 	1    9200 4850
@@
 F 0 "LD7" H 9193 5145 50  0000 C CNN
 F 1 "Green" H 9193 5236 50  0000 C CNN
-F 2 "" H 9200 5400 50  0001 C CNN
+F 2 "footprints:LED_0603" H 9200 5400 50  0001 C CNN
 F 3 "~" H 9200 5400 50  0001 C CNN
 	1    9200 5400
@@
 F 0 "R17" V 8393 1500 50  0000 C CNN
 F 1 "2K2±5% 0.063W" V 8484 1500 50  0000 C CNN
-F 2 "" V 8530 1500 50  0001 C CNN
+F 2 "footprints:R_Array_Convex_4x0603" V 8530 1500 50  0001 C CNN
 F 3 "~" H 8600 1500 50  0001 C CNN
 	1    8600 1500
@@
 F 0 "R18" V 8393 2000 50  0000 C CNN
 F 1 "2K2±5% 0.063W" V 8484 2000 50  0000 C CNN
-F 2 "" V 8530 2000 50  0001 C CNN
+F 2 "footprints:R_Array_Convex_4x0603" V 8530 2000 50  0001 C CNN
 F 3 "~" H 8600 2000 50  0001 C CNN
 	1    8600 2000
@@
 F 0 "R40" V 8393 2550 50  0000 C CNN
 F 1 "2K2±5% 0.063W" V 8484 2550 50  0000 C CNN
-F 2 "" V 8530 2550 50  0001 C CNN
+F 2 "footprints:R_0402" V 8530 2550 50  0001 C CNN
 F 3 "~" H 8600 2550 50  0001 C CNN
 	1    8600 2550
@@
 F 0 "R41" V 8393 3100 50  0000 C CNN
 F 1 "2K2±5% 0.063W" V 8484 3100 50  0000 C CNN
-F 2 "" V 8530 3100 50  0001 C CNN
+F 2 "footprints:R_0402" V 8530 3100 50  0001 C CNN
 F 3 "~" H 8600 3100 50  0001 C CNN
 	1    8600 3100
@@
 F 0 "R42" V 8393 3700 50  0000 C CNN
 F 1 "2K2±5% 0.063W" V 8484 3700 50  0000 C CNN
-F 2 "" V 8530 3700 50  0001 C CNN
+F 2 "footprints:R_0402" V 8530 3700 50  0001 C CNN
 F 3 "~" H 8600 3700 50  0001 C CNN
 	1    8600 3700
@@
 F 0 "R43" V 8393 4300 50  0000 C CNN
 F 1 "2K2±5% 0.063W" V 8484 4300 50  0000 C CNN
-F 2 "" V 8530 4300 50  0001 C CNN
+F 2 "footprints:R_0402" V 8530 4300 50  0001 C CNN
 F 3 "~" H 8600 4300 50  0001 C CNN
 	1    8600 4300
@@
 F 0 "R44" V 8393 4850 50  0000 C CNN
 F 1 "2K2±5% 0.063W" V 8484 4850 50  0000 C CNN
-F 2 "" V 8530 4850 50  0001 C CNN
+F 2 "footprints:R_0402" V 8530 4850 50  0001 C CNN
 F 3 "~" H 8600 4850 50  0001 C CNN
 	1    8600 4850
@@
 F 0 "R45" V 8393 5400 50  0000 C CNN
 F 1 "2K2±5% 0.063W" V 8484 5400 50  0000 C CNN
-F 2 "" V 8530 5400 50  0001 C CNN
+F 2 "footprints:R_0402" V 8530 5400 50  0001 C CNN
 F 3 "~" H 8600 5400 50  0001 C CNN
 	1    8600 5400
@@
 F 0 "U7" H 3675 3099 60  0000 C CNN
 F 1 "ADS7924" H 3675 2993 60  0000 C CNN
-F 2 "" H 3120 2910 60  0001 C CNN
+F 2 "footprints:QFN16" H 3120 2910 60  0001 C CNN
 F 3 "" H 3120 2910 60  0000 C CNN
 	1    2900 2800
@@
 F 0 "J17" H 2343 4111 60  0000 C CNN
 F 1 "1x4_male_pin_Header_2.54mm" H 2340 3460 60  0001 C CNN
-F 2 "" H 2450 4200 60  0001 C CNN
+F 2 "footprints:1x04-pin-header-2.54mm" H 2450 4200 60  0001 C CNN
 F 3 "" H 2450 4200 60  0000 C CNN
 	1    2450 3650
@@
 F 0 "J15" H 1743 4111 60  0000 C CNN
 F 1 "1x4_male_pin_Header_2.54mm" H 1740 3460 60  0001 C CNN
-F 2 "" H 1850 4200 60  0001 C CNN
+F 2 "footprints:1x04-pin-header-2.54mm" H 1850 4200 60  0001 C CNN
 F 3 "" H 1850 4200 60  0000 C CNN
 	1    1850 3650
@@
 F 0 "J16" H 1093 4111 60  0000 C CNN
 F 1 "1x4_male_pin_Header_2.54mm" H 1090 3460 60  0001 C CNN
-F 2 "" H 1200 4200 60  0001 C CNN
+F 2 "footprints:1x04-pin-header-2.54mm" H 1200 4200 60  0001 C CNN
 F 3 "" H 1200 4200 60  0000 C CNN
 	1    1200 3650
@@
 F 0 "C46" V 2998 1900 50  0000 C CNN
 F 1 "100 nF" V 3089 1900 50  0000 C CNN
-F 2 "" H 3288 1750 50  0001 C CNN
+F 2 "footprints:C_0402" H 3288 1750 50  0001 C CNN
 F 3 "~" H 3250 1900 50  0001 C CNN
 	1    3250 1900
@@
 F 0 "C45" V 3898 1900 50  0000 C CNN
 F 1 "100 nF" V 3989 1900 50  0000 C CNN
-F 2 "" H 4188 1750 50  0001 C CNN
+F 2 "footprints:C_0402" H 4188 1750 50  0001 C CNN
 F 3 "~" H 4150 1900 50  0001 C CNN
 	1    4150 1900
@@
 F 0 "R19" V 2093 1900 50  0000 C CNN
 F 1 "10K±5% 0.063W" V 2184 1900 50  0000 C CNN
-F 2 "" V 2230 1900 50  0001 C CNN
+F 2 "footprints:R_0402" V 2230 1900 50  0001 C CNN
 F 3 "~" H 2300 1900 50  0001 C CNN
 	1    2300 1900
@@
 F 0 "R20" H 4880 2454 50  0000 R CNN
 F 1 "10K±5% 0.063W" V 5050 2800 50  0000 R CNN
-F 2 "" V 4880 2500 50  0001 C CNN
+F 2 "footprints:R_0402" V 4880 2500 50  0001 C CNN
 F 3 "~" H 4950 2500 50  0001 C CNN
 	1    4950 2500
@@
 F 0 "R21" H 5330 2454 50  0000 R CNN
 F 1 "10K±5% 0.063W" V 5500 2800 50  0000 R CNN
-F 2 "" V 5330 2500 50  0001 C CNN
+F 2 "footprints:R_0402" V 5330 2500 50  0001 C CNN
 F 3 "~" H 5400 2500 50  0001 C CNN
 	1    5400 2500
@@
 F 0 "JP1" V 1753 915 60  0000 R CNN
 F 1 "Jumper_3pin" V 1647 915 60  0000 R CNN
-F 2 "" H 1750 1000 60  0001 C CNN
+F 2 "footprints:1x03-pin-header-2.54mm" H 1750 1000 60  0001 C CNN
 F 3 "" H 1750 1000 60  0000 C CNN
 	1    1850 1000
@@
 F 0 "SW1" H 4575 5743 60  0000 C CNN
 F 1 "SW1" H 4575 5743 60  0001 C CNN
-F 2 "" H 4200 5550 60  0001 C CNN
+F 2 "footprints:SW_SMD_60X3.8" H 4200 5550 60  0001 C CNN
 F 3 "" H 4200 5550 60  0000 C CNN
 	1    4200 5550
@@
 F 0 "SW2" H 4625 6843 60  0000 C CNN
 F 1 "Switch_4p" H 4625 6843 60  0001 C CNN
-F 2 "" H 4250 6650 60  0001 C CNN
+F 2 "footprints:SW_SMD_60X3.8" H 4250 6650 60  0001 C CNN
 F 3 "" H 4250 6650 60  0000 C CNN
 	1    4250 6650
@@
 F 0 "R31" H 3720 5746 50  0000 L CNN
 F 1 "10K±5% 0.063W" H 3720 5655 50  0000 L CNN
-F 2 "" V 3580 5700 50  0001 C CNN
+F 2 "footprints:R_0402" V 3580 5700 50  0001 C CNN
 F 3 "~" H 3650 5700 50  0001 C CNN
 	1    3650 5700
@@
 F 0 "R32" H 3720 6846 50  0000 L CNN
 F 1 "10K±5% 0.063W" H 3720 6755 50  0000 L CNN
-F 2 "" V 3580 6800 50  0001 C CNN
+F 2 "footprints:R_0402" V 3580 6800 50  0001 C CNN
 F 3 "~" H 3650 6800 50  0001 C CNN
 	1    3650 6800
@@
 F 0 "C35" H 3265 6846 50  0000 L CNN
 F 1 "100 nF" H 3265 6755 50  0000 L CNN
-F 2 "" H 3188 6650 50  0001 C CNN
+F 2 "footprints:C_0402" H 3188 6650 50  0001 C CNN
 F 3 "~" H 3150 6800 50  0001 C CNN
 	1    3150 6800
@@
 F 0 "C34" H 3265 5746 50  0000 L CNN
 F 1 "100 nF" H 3265 5655 50  0000 L CNN
-F 2 "" H 3188 5550 50  0001 C CNN
+F 2 "footprints:C_0402" H 3188 5550 50  0001 C CNN
 F 3 "~" H 3150 5700 50  0001 C CNN
 	1    3150 5700

Commit message: se coloco hojas de datos de los componentes
Changed lines of the file:
@@
 F 1 "ADS7924" H 3675 2993 60  0000 C CNN
 F 2 "footprints:QFN16" H 3120 2910 60  0001 C CNN
-F 3 "" H 3120 2910 60  0000 C CNN
+F 3 "ads7924.pdf" H 4000 1500 60  0000 C CNN
 	1    2900 2800
 	1    0    0    -1

Commit message: se realizo las correcciones sugeridas por el revisor
Other:
- note added: "Polarized Output Leds"
- note added: "Switch buttons 1 and 2"
Changed lines of the file:
@@
 Wire Wire Line
 	1650 800  1650 1000
+Wire Notes Line
+	7550 1100 7550 6050
+Wire Notes Line
+	7550 6050 9950 6050
+Wire Notes Line
+	9950 6050 9950 1100
+Wire Notes Line
+	9950 1100 7550 1100
+Text Notes 7550 1050 0    129  ~ 26
+Polarized Output Leds
+Wire Notes Line
+	6050 4950 6050 7500
+Wire Notes Line
+	6050 7500 2350 7500
+Wire Notes Line
+	2350 7500 2350 4950
+Wire Notes Line
+	2350 4950 6050 4950
+Text Notes 3000 4850 0    129  ~ 26
+Switch buttons 1 and 2
 $EndSCHEMATC
