File: FPGA_Lattice_Replica_Icezum/USB_communication.sch (KiCad schematic (older format))
At the start: 38 parts, among them J1 USB_Micro_Type_B, U3 FT2232H, U4 DSC1001, U5 93LC56C

Commit message: se mejoro esquematico de acuerdo a la revisión del docente. Se mejoro rotulo (se coloco link del repo, autor y autor de la versión original y la licencia) se mejoro el flujo izquiera derecha de los botones, se desplazo fiduciales a la página principal, se achico el esquematico en la parte de headers
Parts:
- C17, C22, C24, C31, C32: footprint footprints:C_0603 -> footprints:L_0805
- C18, C19, C20, C21, C23, C25, C26, C27, C28, C29, C30, C33: footprint footprints:C_0402 -> footprints:L_0805
- R10, R11, R12, R13, R14, R15, R16, R47, R48: footprint footprints:R_0402 -> footprints:F_0805
Changed lines of the file:
@@
 Comp "Especialización en Sistemas Embebidos - DCI (7 Cohorte )"
 Comment1 "Proyecto para trabajo final de la materia DCI - CESE-7Co2018"
-Comment2 "Revisor del trabajo: Gustavo Paredes Delayone"
-Comment3 "Revisor suplente : Rafael Oliva curso CESE en la 6 Cohorte"
-Comment4 ""
+Comment2 "Revisores del trabajo: Gustavo Paredes Delayone, Rafael Oliva curso CESE en la 6 Cohorte"
+Comment3 "License: Creative commons Attribution ShareAlike"
+Comment4 "Autor: Jacobo O. Salvador. Adaptador versión  original (Eladio Delgado Mingorance)"
 $EndDescr
 $Comp
@@
 F 0 "C33" H 7415 5846 50  0000 L CNN
 F 1 "100 nF" H 7415 5755 50  0000 L CNN
-F 2 "footprints:C_0402" H 7338 5650 50  0001 C CNN
+F 2 "footprints:L_0805" H 7338 5650 50  0001 C CNN
 F 3 "~" H 7300 5800 50  0001 C CNN
 	1    7300 5800
@@
 F 0 "R12" H 9370 5146 50  0000 L CNN
 F 1 "10K±5% 0.063W" V 9200 4800 50  0000 L CNN
-F 2 "footprints:R_0402" V 9230 5100 50  0001 C CNN
+F 2 "footprints:F_0805" V 9230 5100 50  0001 C CNN
 F 3 "~" H 9300 5100 50  0001 C CNN
 	1    9300 5100
@@
 F 0 "R13" H 9770 5146 50  0000 L CNN
 F 1 "10K±5% 0.063W" V 9600 4800 50  0000 L CNN
-F 2 "footprints:R_0402" V 9630 5100 50  0001 C CNN
+F 2 "footprints:F_0805" V 9630 5100 50  0001 C CNN
 F 3 "~" H 9700 5100 50  0001 C CNN
 	1    9700 5100
@@
 F 0 "R14" H 10220 5146 50  0000 L CNN
 F 1 "10K±5% 0.063W" V 10050 4800 50  0000 L CNN
-F 2 "footprints:R_0402" V 10080 5100 50  0001 C CNN
+F 2 "footprints:F_0805" V 10080 5100 50  0001 C CNN
 F 3 "~" H 10150 5100 50  0001 C CNN
 	1    10150 5100
@@
 F 0 "C22" V 8798 2300 50  0000 C CNN
 F 1 "10 nF" V 8889 2300 50  0000 C CNN
-F 2 "footprints:C_0603" H 9088 2150 50  0001 C CNN
+F 2 "footprints:L_0805" H 9088 2150 50  0001 C CNN
 F 3 "~" H 9050 2300 50  0001 C CNN
 	1    9050 2300
@@
 F 0 "C23" V 8798 2900 50  0000 C CNN
 F 1 "100 nF" V 8889 2900 50  0000 C CNN
-F 2 "footprints:C_0402" H 9088 2750 50  0001 C CNN
+F 2 "footprints:L_0805" H 9088 2750 50  0001 C CNN
 F 3 "~" H 9050 2900 50  0001 C CNN
 	1    9050 2900
@@
 F 0 "C26" H 4215 2396 50  0000 L CNN
 F 1 "100 nF" H 4215 2305 50  0000 L CNN
-F 2 "footprints:C_0402" H 4138 2200 50  0001 C CNN
+F 2 "footprints:L_0805" H 4138 2200 50  0001 C CNN
 F 3 "~" H 4100 2350 50  0001 C CNN
 	1    4100 2350
@@
 F 0 "C27" H 4815 2396 50  0000 L CNN
 F 1 "100 nF" H 4815 2305 50  0000 L CNN
-F 2 "footprints:C_0402" H 4738 2200 50  0001 C CNN
+F 2 "footprints:L_0805" H 4738 2200 50  0001 C CNN
 F 3 "~" H 4700 2350 50  0001 C CNN
 	1    4700 2350
@@
 F 0 "C28" H 5415 2396 50  0000 L CNN
 F 1 "100 nF" H 5415 2305 50  0000 L CNN
-F 2 "footprints:C_0402" H 5338 2200 50  0001 C CNN
+F 2 "footprints:L_0805" H 5338 2200 50  0001 C CNN
 F 3 "~" H 5300 2350 50  0001 C CNN
 	1    5300 2350
@@
 F 0 "C29" H 6065 2396 50  0000 L CNN
 F 1 "100 nF" H 6065 2305 50  0000 L CNN
-F 2 "footprints:C_0402" H 5988 2200 50  0001 C CNN
+F 2 "footprints:L_0805" H 5988 2200 50  0001 C CNN
 F 3 "~" H 5950 2350 50  0001 C CNN
 	1    5950 2350
@@
 F 0 "C19" H 3665 1596 50  0000 L CNN
 F 1 "100 nF" H 3665 1505 50  0000 L CNN
-F 2 "footprints:C_0402" H 3588 1400 50  0001 C CNN
+F 2 "footprints:L_0805" H 3588 1400 50  0001 C CNN
 F 3 "~" H 3550 1550 50  0001 C CNN
 	1    3550 1550
@@
 F 0 "C20" H 4215 1596 50  0000 L CNN
 F 1 "100 nF" H 4215 1505 50  0000 L CNN
-F 2 "footprints:C_0402" H 4138 1400 50  0001 C CNN
+F 2 "footprints:L_0805" H 4138 1400 50  0001 C CNN
 F 3 "~" H 4100 1550 50  0001 C CNN
 	1    4100 1550
@@
 F 0 "C21" H 4765 1596 50  0000 L CNN
 F 1 "100 nF" H 4765 1505 50  0000 L CNN
-F 2 "footprints:C_0402" H 4688 1400 50  0001 C CNN
+F 2 "footprints:L_0805" H 4688 1400 50  0001 C CNN
 F 3 "~" H 4650 1550 50  0001 C CNN
 	1    4650 1550
@@
 F 0 "C25" H 2815 2396 50  0000 L CNN
 F 1 "100 nF" H 2815 2305 50  0000 L CNN
-F 2 "footprints:C_0402" H 2738 2200 50  0001 C CNN
+F 2 "footprints:L_0805" H 2738 2200 50  0001 C CNN
 F 3 "~" H 2700 2350 50  0001 C CNN
 	1    2700 2350
@@
 F 0 "C24" H 2315 2396 50  0000 L CNN
 F 1 "4.7 uF" H 2315 2305 50  0000 L CNN
-F 2 "footprints:C_0603" H 2238 2200 50  0001 C CNN
+F 2 "footprints:L_0805" H 2238 2200 50  0001 C CNN
 F 3 "~" H 2200 2350 50  0001 C CNN
 	1    2200 2350
@@
 F 0 "C18" H 2815 1596 50  0000 L CNN
 F 1 "100 nF" H 2815 1505 50  0000 L CNN
-F 2 "footprints:C_0402" H 2738 1400 50  0001 C CNN
+F 2 "footprints:L_0805" H 2738 1400 50  0001 C CNN
 F 3 "~" H 2700 1550 50  0001 C CNN
 	1    2700 1550
@@
 F 0 "C17" H 2315 1596 50  0000 L CNN
 F 1 "4.7 uF" H 2315 1505 50  0000 L CNN
-F 2 "footprints:C_0603" H 2238 1400 50  0001 C CNN
+F 2 "footprints:L_0805" H 2238 1400 50  0001 C CNN
 F 3 "~" H 2200 1550 50  0001 C CNN
 	1    2200 1550
@@
 F 0 "C31" H 1815 3846 50  0000 L CNN
 F 1 "4.7 uF" H 1815 3755 50  0000 L CNN
-F 2 "footprints:C_0603" H 1738 3650 50  0001 C CNN
+F 2 "footprints:L_0805" H 1738 3650 50  0001 C CNN
 F 3 "~" H 1700 3800 50  0001 C CNN
 	1    1700 3800
@@
 F 0 "R48" H 5650 6550 50  0000 L CNN
 F 1 "2K2±5% 0.063W" H 5600 6400 50  0000 L CNN
-F 2 "footprints:R_0402" V 5530 6550 50  0001 C CNN
+F 2 "footprints:F_0805" V 5530 6550 50  0001 C CNN
 F 3 "~" H 5600 6550 50  0001 C CNN
 	1    5600 6550
@@
 F 0 "R47" H 6350 6550 50  0000 L CNN
 F 1 "2K2±5% 0.063W" H 6300 6400 50  0000 L CNN
-F 2 "footprints:R_0402" V 6230 6550 50  0001 C CNN
+F 2 "footprints:F_0805" V 6230 6550 50  0001 C CNN
 F 3 "~" H 6300 6550 50  0001 C CNN
 	1    6300 6550
@@
 F 0 "C32" H 1465 5746 50  0000 L CNN
 F 1 "10 nF" H 1465 5655 50  0000 L CNN
-F 2 "footprints:C_0603" H 1388 5550 50  0001 C CNN
+F 2 "footprints:L_0805" H 1388 5550 50  0001 C CNN
 F 3 "~" H 1350 5700 50  0001 C CNN
 	1    1350 5700
@@
 F 0 "R11" H 2030 5054 50  0000 R CNN
 F 1 "12K±1% 0.063W" V 2250 5500 50  0000 R CNN
-F 2 "footprints:R_0402" V 2030 5100 50  0001 C CNN
+F 2 "footprints:F_0805" V 2030 5100 50  0001 C CNN
 F 3 "~" H 2100 5100 50  0001 C CNN
 	1    2100 5100
@@
 F 0 "R10" H 1320 4596 50  0000 L CNN
 F 1 "2K2±5% 0.063W" H 1320 4505 50  0000 L CNN
-F 2 "footprints:R_0402" V 1180 4550 50  0001 C CNN
+F 2 "footprints:F_0805" V 1180 4550 50  0001 C CNN
 F 3 "~" H 1250 4550 50  0001 C CNN
 	1    1250 4550
@@
 F 0 "C30" H 1265 3596 50  0000 L CNN
 F 1 "100 nF" H 1265 3505 50  0000 L CNN
-F 2 "footprints:C_0402" H 1188 3400 50  0001 C CNN
+F 2 "footprints:L_0805" H 1188 3400 50  0001 C CNN
 F 3 "~" H 1150 3550 50  0001 C CNN
 	1    1150 3550
@@
 F 0 "R16" V 1750 7050 50  0000 C CNN
 F 1 "0R±5% 0.063W" V 1950 7050 50  0000 C CNN
-F 2 "footprints:R_0402" V 1780 7050 50  0001 C CNN
+F 2 "footprints:F_0805" V 1780 7050 50  0001 C CNN
 F 3 "~" H 1850 7050 50  0001 C CNN
 	1    1850 7050
@@
 F 0 "R15" V 10400 6000 50  0000 L CNN
 F 1 "2K2±5% 0.063W" V 10200 5750 50  0000 L CNN
-F 2 "footprints:R_0402" V 10230 6050 50  0001 C CNN
+F 2 "footprints:F_0805" V 10230 6050 50  0001 C CNN
 F 3 "~" H 10300 6050 50  0001 C CNN
 	1    10300 6050
